File: v2/kicad/rgb-led-v2.sch (KiCad schematic (older format))
At the start: 8 parts, among them U1 ARDUINO_NANO

Commit message: Continued work on v2
Parts:
- added SW1: SWITCH_INV, ~, symbol SWITCH_INV
- renumbered CONN_4 to CONN1, QB to QB1, QG to QG1, QR to QR1, U1 to UC1
Connections:
- wire segments 48 -> 49
- no-connect marks 0 -> 21
Other:
- moved on the sheet: CONN1, QB1, QG1, QR1, RV1, RV2, RV3

Commit message: Continued work on v2
Parts:
- removed SW1: SWITCH_INV, ~, symbol SWITCH_INV
- added SW1: SPST, ~, symbol SPST
Connections:
- no-connect marks 21 -> 20
Changed lines of the file:
@@
 LIBS:valves
 LIBS:arduino-nano
-LIBS:rgb-led-v2-cache
 EELAYER 27 0
 EELAYER END
@@
 Sheet 1 1
 Title "RGB LED v2"
-Date "27 nov 2014"
+Date "28 nov 2014"
 Rev "1"
 Comp "coredump Hackerspace"
@@
 $Comp
 L PWR_FLAG #FLG05
-U 1 1 5477A74A
-P 3250 750
-F 0 "#FLG05" H 3250 845 30  0001 C CNN
-F 1 "PWR_FLAG" H 3250 930 30  0000 C CNN
-F 2 "" H 3250 750 60  0000 C CNN
-F 3 "" H 3250 750 60  0000 C CNN
-	1    3250 750
-	1    0    0    -1
-$EndComp
-$Comp
-L PWR_FLAG #FLG06
 U 1 1 5477A759
 P 3500 4200
-F 0 "#FLG06" H 3500 4295 30  0001 C CNN
+F 0 "#FLG05" H 3500 4295 30  0001 C CNN
 F 1 "PWR_FLAG" H 3500 4380 30  0000 C CNN
 F 2 "" H 3500 4200 60  0000 C CNN
@@
 NoConn ~ 3550 1500
 NoConn ~ 2700 3850
-$Comp
-L SWITCH_INV SW1
-U 1 1 5477A860
-P 2100 850
-F 0 "SW1" H 1900 1000 50  0000 C CNN
-F 1 "SWITCH_INV" H 1950 700 50  0000 C CNN
-F 2 "~" H 2100 850 60  0000 C CNN
-F 3 "~" H 2100 850 60  0000 C CNN
-	1    2100 850
-	1    0    0    -1
-$EndComp
 Wire Wire Line
 	3400 1350 3400 1500
@@
 	6600 1900 5800 1900
 Wire Wire Line
-	6900 750  6900 1950
+	6900 850  6900 1950
 Wire Wire Line
 	4850 1700 4850 1800
@@
 	950  850  1600 850
 Wire Wire Line
-	3250 750  3250 1500
-NoConn ~ 2600 950
-Wire Wire Line
-	2600 750  6900 750
-Connection ~ 3250 750
-$Comp
-L PWR_FLAG #FLG07
+	3250 850  3250 1500
+Wire Wire Line
+	2600 850  6900 850
+$Comp
+L PWR_FLAG #FLG06
 U 1 1 5477AA91
 P 1200 800
-F 0 "#FLG07" H 1200 895 30  0001 C CNN
+F 0 "#FLG06" H 1200 895 30  0001 C CNN
 F 1 "PWR_FLAG" H 1200 980 30  0000 C CNN
 F 2 "" H 1200 800 60  0000 C CNN
@@
 Connection ~ 1200 850
 $Comp
-L GND #PWR08
+L GND #PWR07
 U 1 1 5477A965
 P 1900 3300
-F 0 "#PWR08" H 1900 3300 30  0001 C CNN
+F 0 "#PWR07" H 1900 3300 30  0001 C CNN
 F 1 "GND" H 1900 3230 30  0001 C CNN
 F 2 "" H 1900 3300 60  0000 C CNN
@@
 $EndComp
 $Comp
-L GND #PWR09
+L GND #PWR08
 U 1 1 5477A96B
 P 1900 2800
-F 0 "#PWR09" H 1900 2800 30  0001 C CNN
+F 0 "#PWR08" H 1900 2800 30  0001 C CNN
 F 1 "GND" H 1900 2730 30  0001 C CNN
 F 2 "" H 1900 2800 60  0000 C CNN
@@
 $EndComp
 $Comp
-L GND #PWR010
+L GND #PWR09
 U 1 1 5477A971
 P 1900 2300
-F 0 "#PWR010" H 1900 2300 30  0001 C CNN
+F 0 "#PWR09" H 1900 2300 30  0001 C CNN
 F 1 "GND" H 1900 2230 30  0001 C CNN
 F 2 "" H 1900 2300 60  0000 C CNN
@@
 	1900 3200 1900 3300
 $Comp
-L GND #PWR011
+L GND #PWR010
 U 1 1 5477AAB7
 P 3400 4200
-F 0 "#PWR011" H 3400 4200 30  0001 C CNN
+F 0 "#PWR010" H 3400 4200 30  0001 C CNN
 F 1 "GND" H 3400 4130 30  0001 C CNN
 F 2 "" H 3400 4200 60  0000 C CNN
@@
 Wire Wire Line
 	1900 2200 1550 2200
+$Comp
+L SPST SW1
+U 1 1 547836EC
+P 2100 850
+F 0 "SW1" H 2100 950 70  0000 C CNN
+F 1 "SPST" H 2100 750 70  0000 C CNN
+F 2 "~" H 2100 850 60  0000 C CNN
+F 3 "~" H 2100 850 60  0000 C CNN
+	1    2100 850
+	1    0    0    -1
+$EndComp
+$Comp
+L PWR_FLAG #FLG011
+U 1 1 547837AB
+P 3250 850
+F 0 "#FLG011" H 3250 945 30  0001 C CNN
+F 1 "PWR_FLAG" H 3250 1030 30  0000 C CNN
+F 2 "" H 3250 850 60  0000 C CNN
+F 3 "" H 3250 850 60  0000 C CNN
+	1    3250 850
+	1    0    0    -1
+$EndComp
 $EndSCHEMATC

Commit message: [v2] Finished netlist assignment
Parts:
- added CONN2: VCC 12V, ~, symbol CONN_2
Connections:
- net labels removed: +12V
- wire segments 49 -> 51
Changed lines of the file:
@@
 LIBS:valves
 LIBS:arduino-nano
+LIBS:rgb-led-v2-cache
 EELAYER 27 0
 EELAYER END
@@
 Sheet 1 1
 Title "RGB LED v2"
-Date "28 nov 2014"
+Date "29 nov 2014"
 Rev "1"
 Comp "coredump Hackerspace"
@@
 	1    5650 2250
 	1    0    0    -1
-$EndComp
-$Comp
-L +12V #PWR01
-U 1 1 5476D52F
-P 950 850
-F 0 "#PWR01" H 950 800 20  0001 C CNN
-F 1 "+12V" H 950 950 30  0000 C CNN
-F 2 "" H 950 850 60  0000 C CNN
-F 3 "" H 950 850 60  0000 C CNN
-	1    950  850
-	0    -1   -1   0
 $EndComp
 $Comp
@@
 $EndComp
 $Comp
-L GND #PWR02
+L GND #PWR01
 U 1 1 5477A4E7
 P 4850 1800
-F 0 "#PWR02" H 4850 1800 30  0001 C CNN
+F 0 "#PWR01" H 4850 1800 30  0001 C CNN
 F 1 "GND" H 4850 1730 30  0001 C CNN
 F 2 "" H 4850 1800 60  0000 C CNN
@@
 $EndComp
 $Comp
-L GND #PWR03
+L GND #PWR02
 U 1 1 5477A4F4
 P 4850 2700
-F 0 "#PWR03" H 4850 2700 30  0001 C CNN
+F 0 "#PWR02" H 4850 2700 30  0001 C CNN
 F 1 "GND" H 4850 2630 30  0001 C CNN
 F 2 "" H 4850 2700 60  0000 C CNN
@@
 $EndComp
 $Comp
-L GND #PWR04
+L GND #PWR03
 U 1 1 5477A4FA
 P 4850 3600
-F 0 "#PWR04" H 4850 3600 30  0001 C CNN
+F 0 "#PWR03" H 4850 3600 30  0001 C CNN
 F 1 "GND" H 4850 3530 30  0001 C CNN
 F 2 "" H 4850 3600 60  0000 C CNN
@@
 $EndComp
 $Comp
-L PWR_FLAG #FLG05
+L PWR_FLAG #FLG04
 U 1 1 5477A759
 P 3500 4200
-F 0 "#FLG05" H 3500 4295 30  0001 C CNN
+F 0 "#FLG04" H 3500 4295 30  0001 C CNN
 F 1 "PWR_FLAG" H 3500 4380 30  0000 C CNN
 F 2 "" H 3500 4200 60  0000 C CNN
@@
 	4850 3500 4850 3600
 Wire Wire Line
-	950  850  1600 850
+	1050 850  1600 850
 Wire Wire Line
 	3250 850  3250 1500
@@
 	2600 850  6900 850
 $Comp
-L PWR_FLAG #FLG06
+L PWR_FLAG #FLG05
 U 1 1 5477AA91
 P 1200 800
-F 0 "#FLG06" H 1200 895 30  0001 C CNN
+F 0 "#FLG05" H 1200 895 30  0001 C CNN
 F 1 "PWR_FLAG" H 1200 980 30  0000 C CNN
 F 2 "" H 1200 800 60  0000 C CNN
@@
 Connection ~ 1200 850
 $Comp
-L GND #PWR07
+L GND #PWR06
 U 1 1 5477A965
 P 1900 3300
-F 0 "#PWR07" H 1900 3300 30  0001 C CNN
+F 0 "#PWR06" H 1900 3300 30  0001 C CNN
 F 1 "GND" H 1900 3230 30  0001 C CNN
 F 2 "" H 1900 3300 60  0000 C CNN
@@
 $EndComp
 $Comp
-L GND #PWR08
+L GND #PWR07
 U 1 1 5477A96B
 P 1900 2800
-F 0 "#PWR08" H 1900 2800 30  0001 C CNN
+F 0 "#PWR07" H 1900 2800 30  0001 C CNN
 F 1 "GND" H 1900 2730 30  0001 C CNN
 F 2 "" H 1900 2800 60  0000 C CNN
@@
 $EndComp
 $Comp
-L GND #PWR09
+L GND #PWR08
 U 1 1 5477A971
 P 1900 2300
-F 0 "#PWR09" H 1900 2300 30  0001 C CNN
+F 0 "#PWR08" H 1900 2300 30  0001 C CNN
 F 1 "GND" H 1900 2230 30  0001 C CNN
 F 2 "" H 1900 2300 60  0000 C CNN
@@
 	1900 3200 1900 3300
 $Comp
-L GND #PWR010
+L GND #PWR09
 U 1 1 5477AAB7
 P 3400 4200
-F 0 "#PWR010" H 3400 4200 30  0001 C CNN
+F 0 "#PWR09" H 3400 4200 30  0001 C CNN
 F 1 "GND" H 3400 4130 30  0001 C CNN
 F 2 "" H 3400 4200 60  0000 C CNN
@@
 $EndComp
 $Comp
-L PWR_FLAG #FLG011
+L PWR_FLAG #FLG010
 U 1 1 547837AB
 P 3250 850
-F 0 "#FLG011" H 3250 945 30  0001 C CNN
+F 0 "#FLG010" H 3250 945 30  0001 C CNN
 F 1 "PWR_FLAG" H 3250 1030 30  0000 C CNN
 F 2 "" H 3250 850 60  0000 C CNN
@@
 	1    0    0    -1
 $EndComp
+$Comp
+L CONN_2 CONN2
+U 1 1 547A1B2B
+P 700 950
+F 0 "CONN2" V 650 950 40  0000 C CNN
+F 1 "VCC 12V" V 750 950 40  0000 C CNN
+F 2 "~" H 700 950 60  0000 C CNN
+F 3 "~" H 700 950 60  0000 C CNN
+	1    700  950
+	-1   0    0    -1
+$EndComp
+$Comp
+L GND #PWR011
+U 1 1 547A1B66
+P 1200 1150
+F 0 "#PWR011" H 1200 1150 30  0001 C CNN
+F 1 "GND" H 1200 1080 30  0001 C CNN
+F 2 "" H 1200 1150 60  0000 C CNN
+F 3 "" H 1200 1150 60  0000 C CNN
+	1    1200 1150
+	1    0    0    -1
+$EndComp
+Wire Wire Line
+	1050 1050 1200 1050
+Wire Wire Line
+	1200 1050 1200 1150
 $EndSCHEMATC

Commit message: [v2] Started work on PCB layout
Connections:
- net labels added: gnd
Changed lines of the file:
@@
-$EndComp
-$Comp
-L GND #PWR03
-U 1 1 5477A4FA
-P 4850 3600
-F 0 "#PWR03" H 4850 3600 30  0001 C CNN
-F 1 "GND" H 4850 3530 30  0001 C CNN
-F 2 "" H 4850 3600 60  0000 C CNN
-F 3 "" H 4850 3600 60  0000 C CNN
-	1    4850 3600
-	1    0    0    -1
 $EndComp
 $Comp
@@
 	5800 2600 4850 2600
 Wire Wire Line
-	5800 3500 4850 3500
-Wire Wire Line
 	6900 2050 6700 2050
 Wire Wire Line
@@
 Wire Wire Line
 	4850 2600 4850 2700
-Wire Wire Line
-	4850 3500 4850 3600
 Wire Wire Line
 	1050 850  1600 850
@@
 Wire Wire Line
 	1200 1050 1200 1150
+Wire Wire Line
+	4850 3500 4850 3600
+Wire Wire Line
+	5800 3500 4850 3500
+$Comp
+L GND #PWR03
+U 1 1 5477A4FA
+P 4850 3600
+F 0 "#PWR03" H 4850 3600 30  0001 C CNN
+F 1 "GND" H 4850 3530 30  0001 C CNN
+F 2 "" H 4850 3600 60  0000 C CNN
+F 3 "" H 4850 3600 60  0000 C CNN
+	1    4850 3600
+	1    0    0    -1
+$EndComp
+Text Label 5350 3500 0    60   ~ 0
+GND
+Text Label 5400 3500 0    60   ~ 0
+GND
+Text Label 5050 1700 0    60   ~ 0
+GND
+Text Label 5100 2600 0    60   ~ 0
+GND
+Text Label 4850 3600 0    60   ~ 0
+gnd
 $EndSCHEMATC

Commit message: [v2] Configured track widths
Changed lines of the file:
@@
 Sheet 1 1
 Title "RGB LED v2"
-Date "29 nov 2014"
+Date "30 nov 2014"
 Rev "1"
 Comp "coredump Hackerspace"
@@
 $EndComp
 $Comp
-L PWR_FLAG #FLG04
+L PWR_FLAG #FLG03
 U 1 1 5477A759
 P 3500 4200
-F 0 "#FLG04" H 3500 4295 30  0001 C CNN
+F 0 "#FLG03" H 3500 4295 30  0001 C CNN
 F 1 "PWR_FLAG" H 3500 4380 30  0000 C CNN
 F 2 "" H 3500 4200 60  0000 C CNN
@@
 	4850 2600 4850 2700
 Wire Wire Line
-	1050 850  1600 850
+	1050 850  2000 850
 Wire Wire Line
 	3250 850  3250 1500
 Wire Wire Line
-	2600 850  6900 850
-$Comp
-L PWR_FLAG #FLG05
+	3000 850  6900 850
+$Comp
+L PWR_FLAG #FLG04
 U 1 1 5477AA91
 P 1200 800
-F 0 "#FLG05" H 1200 895 30  0001 C CNN
+F 0 "#FLG04" H 1200 895 30  0001 C CNN
 F 1 "PWR_FLAG" H 1200 980 30  0000 C CNN
 F 2 "" H 1200 800 60  0000 C CNN
@@
 $EndComp
 Wire Wire Line
-	1200 800  1200 850
+	1200 850  1200 800
 Connection ~ 1200 850
 $Comp
-L GND #PWR06
+L GND #PWR05
 U 1 1 5477A965
 P 1900 3300
-F 0 "#PWR06" H 1900 3300 30  0001 C CNN
+F 0 "#PWR05" H 1900 3300 30  0001 C CNN
 F 1 "GND" H 1900 3230 30  0001 C CNN
 F 2 "" H 1900 3300 60  0000 C CNN
@@
 $EndComp
 $Comp
-L GND #PWR07
+L GND #PWR06
 U 1 1 5477A96B
 P 1900 2800
-F 0 "#PWR07" H 1900 2800 30  0001 C CNN
+F 0 "#PWR06" H 1900 2800 30  0001 C CNN
 F 1 "GND" H 1900 2730 30  0001 C CNN
 F 2 "" H 1900 2800 60  0000 C CNN
@@
 $EndComp
 $Comp
-L GND #PWR08
+L GND #PWR07
 U 1 1 5477A971
 P 1900 2300
-F 0 "#PWR08" H 1900 2300 30  0001 C CNN
+F 0 "#PWR07" H 1900 2300 30  0001 C CNN
 F 1 "GND" H 1900 2230 30  0001 C CNN
 F 2 "" H 1900 2300 60  0000 C CNN
@@
 	1900 3200 1900 3300
 $Comp
-L GND #PWR09
+L GND #PWR08
 U 1 1 5477AAB7
 P 3400 4200
-F 0 "#PWR09" H 3400 4200 30  0001 C CNN
+F 0 "#PWR08" H 3400 4200 30  0001 C CNN
 F 1 "GND" H 3400 4130 30  0001 C CNN
 F 2 "" H 3400 4200 60  0000 C CNN
@@
 	1900 2200 1550 2200
 $Comp
-L SPST SW1
-U 1 1 547836EC
-P 2100 850
-F 0 "SW1" H 2100 950 70  0000 C CNN
-F 1 "SPST" H 2100 750 70  0000 C CNN
-F 2 "~" H 2100 850 60  0000 C CNN
-F 3 "~" H 2100 850 60  0000 C CNN
-	1    2100 850
-	1    0    0    -1
-$EndComp
-$Comp
-L PWR_FLAG #FLG010
+L PWR_FLAG #FLG09
 U 1 1 547837AB
 P 3250 850
-F 0 "#FLG010" H 3250 945 30  0001 C CNN
+F 0 "#FLG09" H 3250 945 30  0001 C CNN
 F 1 "PWR_FLAG" H 3250 1030 30  0000 C CNN
 F 2 "" H 3250 850 60  0000 C CNN
@@
 $EndComp
 $Comp
-L GND #PWR011
+L GND #PWR010
 U 1 1 547A1B66
 P 1200 1150
-F 0 "#PWR011" H 1200 1150 30  0001 C CNN
+F 0 "#PWR010" H 1200 1150 30  0001 C CNN
 F 1 "GND" H 1200 1080 30  0001 C CNN
 F 2 "" H 1200 1150 60  0000 C CNN
@@
 	5800 3500 4850 3500
 $Comp
-L GND #PWR03
+L GND #PWR011
 U 1 1 5477A4FA
 P 4850 3600
-F 0 "#PWR03" H 4850 3600 30  0001 C CNN
+F 0 "#PWR011" H 4850 3600 30  0001 C CNN
 F 1 "GND" H 4850 3530 30  0001 C CNN
 F 2 "" H 4850 3600 60  0000 C CNN
@@
 Text Label 4850 3600 0    60   ~ 0
 gnd
+$Comp
+L SPST SW1
+U 1 1 547836EC
+P 2500 850
+F 0 "SW1" H 2500 950 70  0000 C CNN
+F 1 "SPST" H 2500 750 70  0000 C CNN
+F 2 "~" H 2500 850 60  0000 C CNN
+F 3 "~" H 2500 850 60  0000 C CNN
+	1    2500 850
+	1    0    0    -1
+$EndComp
 $EndSCHEMATC

Commit message: [v2] Added fuse
Parts:
- added F1: FUSE, ~, symbol FUSE
Connections:
- wire segments 51 -> 52
Changed lines of the file:
@@
 NoConn ~ 3550 1500
 NoConn ~ 2700 3850
-Wire Wire Line
-	3400 1350 3400 1500
-Wire Wire Line
-	900  1350 3400 1350
-Wire Wire Line
-	900  1350 900  3200
-Wire Wire Line
-	900  2200 1050 2200
-Wire Wire Line
-	900  2700 1050 2700
-Connection ~ 900  2200
-Wire Wire Line
-	900  3200 1050 3200
-Connection ~ 900  2700
-Wire Wire Line
-	1550 3200 1900 3200
-Wire Wire Line
-	1550 2700 1900 2700
-Wire Wire Line
-	1300 2350 1300 2450
-Wire Wire Line
-	1300 2450 2700 2450
-Wire Wire Line
-	1300 2850 1300 3000
-Wire Wire Line
-	1300 3000 2200 3000
-Wire Wire Line
-	2200 3000 2200 2550
-Wire Wire Line
-	2200 2550 2700 2550
-Wire Wire Line
-	1300 3350 1300 3500
-Wire Wire Line
-	1300 3500 2350 3500
-Wire Wire Line
-	2350 3500 2350 2650
-Wire Wire Line
-	2350 2650 2700 2650
-Wire Wire Line
-	4100 3150 5350 3150
-Wire Wire Line
-	4100 2950 4500 2950
-Wire Wire Line
-	4500 2950 4500 2250
-Wire Wire Line
-	4500 2250 5350 2250
-Wire Wire Line
-	4100 2700 4400 2700
-Wire Wire Line
-	4400 2700 4400 1350
-Wire Wire Line
-	4400 1350 5350 1350
-Wire Wire Line
-	5800 1700 4850 1700
-Wire Wire Line
-	5800 2600 4850 2600
-Wire Wire Line
-	6900 2050 6700 2050
-Wire Wire Line
-	6700 2050 6700 1000
-Wire Wire Line
-	6700 1000 5800 1000
-Wire Wire Line
-	6900 2150 6700 2150
-Wire Wire Line
-	6700 2150 6700 2800
-Wire Wire Line
-	6700 2800 5800 2800
-Wire Wire Line
-	6900 2250 6600 2250
-Wire Wire Line
-	6600 2250 6600 1900
-Wire Wire Line
-	6600 1900 5800 1900
-Wire Wire Line
-	6900 850  6900 1950
-Wire Wire Line
-	4850 1700 4850 1800
-Wire Wire Line
-	4850 2600 4850 2700
-Wire Wire Line
-	1050 850  2000 850
-Wire Wire Line
-	3250 850  3250 1500
-Wire Wire Line
-	3000 850  6900 850
 $Comp
 L PWR_FLAG #FLG04
@@
 	1    0    0    -1
 $EndComp
-Wire Wire Line
-	1200 850  1200 800
-Connection ~ 1200 850
 $Comp
 L GND #PWR05
@@
 	-1   0    0    -1
 $EndComp
-Wire Wire Line
-	1900 2200 1900 2300
-Wire Wire Line
-	1900 2700 1900 2800
-Wire Wire Line
-	1900 3200 1900 3300
 $Comp
 L GND #PWR08
@@
 	1    0    0    -1
 $EndComp
-Wire Wire Line
-	1900 2200 1550 2200
 $Comp
 L PWR_FLAG #FLG09
@@
 	1    0    0    -1
 $EndComp
-Wire Wire Line
-	1050 1050 1200 1050
-Wire Wire Line
-	1200 1050 1200 1150
-Wire Wire Line
-	4850 3500 4850 3600
-Wire Wire Line
-	5800 3500 4850 3500
 $Comp
 L GND #PWR011
@@
 	1    0    0    -1
 $EndComp
+Wire Wire Line
+	3400 1350 3400 1500
+Wire Wire Line
+	900  1350 3400 1350
+Wire Wire Line
+	900  1350 900  3200
+Wire Wire Line
+	900  2200 1050 2200
+Wire Wire Line
+	900  2700 1050 2700
+Connection ~ 900  2200
+Wire Wire Line
+	900  3200 1050 3200
+Connection ~ 900  2700
+Wire Wire Line
+	1550 3200 1900 3200
+Wire Wire Line
+	1550 2700 1900 2700
+Wire Wire Line
+	1300 2350 1300 2450
+Wire Wire Line
+	1300 2450 2700 2450
+Wire Wire Line
+	1300 2850 1300 3000
+Wire Wire Line
+	1300 3000 2200 3000
+Wire Wire Line
+	2200 3000 2200 2550
+Wire Wire Line
+	2200 2550 2700 2550
+Wire Wire Line
+	1300 3350 1300 3500
+Wire Wire Line
+	1300 3500 2350 3500
+Wire Wire Line
+	2350 3500 2350 2650
+Wire Wire Line
+	2350 2650 2700 2650
+Wire Wire Line
+	4100 3150 5350 3150
+Wire Wire Line
+	4100 2950 4500 2950
+Wire Wire Line
+	4500 2950 4500 2250
+Wire Wire Line
+	4500 2250 5350 2250
+Wire Wire Line
+	4100 2700 4400 2700
+Wire Wire Line
+	4400 2700 4400 1350
+Wire Wire Line
+	4400 1350 5350 1350
+Wire Wire Line
+	5800 1700 4850 1700
+Wire Wire Line
+	5800 2600 4850 2600
+Wire Wire Line
+	6900 2050 6700 2050
+Wire Wire Line
+	6700 2050 6700 1000
+Wire Wire Line
+	6700 1000 5800 1000
+Wire Wire Line
+	6900 2150 6700 2150
+Wire Wire Line
+	6700 2150 6700 2800
+Wire Wire Line
+	6700 2800 5800 2800
+Wire Wire Line
+	6900 2250 6600 2250
+Wire Wire Line
+	6600 2250 6600 1900
+Wire Wire Line
+	6600 1900 5800 1900
+Wire Wire Line
+	6900 850  6900 1950
+Wire Wire Line
+	4850 1700 4850 1800
+Wire Wire Line
+	4850 2600 4850 2700
+Wire Wire Line
+	1050 850  1450 850
+Wire Wire Line
+	3250 850  3250 1500
+Wire Wire Line
+	3000 850  6900 850
+Wire Wire Line
+	1200 850  1200 800
+Connection ~ 1200 850
+Wire Wire Line
+	1900 2200 1900 2300
+Wire Wire Line
+	1900 2700 1900 2800
+Wire Wire Line
+	1900 3200 1900 3300
+Wire Wire Line
+	1900 2200 1550 2200
+Wire Wire Line
+	1050 1050 1200 1050
+Wire Wire Line
+	1200 1050 1200 1150
+Wire Wire Line
+	4850 3500 4850 3600
+Wire Wire Line
+	5800 3500 4850 3500
+Wire Wire Line
+	1950 850  2000 850
+$Comp
+L FUSE F1
+U 1 1 547B0358
+P 1700 850
+F 0 "F1" H 1800 900 40  0000 C CNN
+F 1 "FUSE" H 1600 800 40  0000 C CNN
+F 2 "~" H 1700 850 60  0000 C CNN
+F 3 "~" H 1700 850 60  0000 C CNN
+	1    1700 850
+	1    0    0    -1
+$EndComp

Commit message: [v2] PCB Routing
Changed lines of the file:
@@
 	1    0    0    -1
 $EndComp
+Connection ~ 3250 850
 $EndSCHEMATC
