File: v1/pcb/rgb_led.kicad_pcb (KiCad board)
At the start: 2 copper layers, 62.7 x 45.2 mm, 8 parts, among them P1 CONN_2, P2 CONN_4, SW1 SWITCH_INV

Commit message: Changed color labels to letters only
Other:
- board text added: "B"
- board text added: "G"
- board text added: "R"
- board text removed: "Blue"
- board text removed: "Green"
- board text removed: "Red"
Changed lines of the file:
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@@
     )
   )
-  (gr_text Blue (at 63.5 45.72) (layer B.Mask)
+  (gr_text B (at 63.5 45.72) (layer B.Mask)
     (effects (font (size 1.5 1.5) (thickness 0.3)) (justify mirror))
   )
-  (gr_text Red (at 45.72 45.72) (layer B.Mask)
+  (gr_text R (at 45.72 45.72) (layer B.Mask)
     (effects (font (size 1.5 1.5) (thickness 0.3)) (justify mirror))
   )
-  (gr_text Green (at 27.94 45.72) (layer B.Mask)
+  (gr_text G (at 27.94 45.72) (layer B.Mask)
     (effects (font (size 1.5 1.5) (thickness 0.3)) (justify mirror))
   )

Commit message: Added OSHW logo
Parts:
- added OSHW_LOGO: , OSHW_COPPER_10MM, F.Cu at (30.5, 19.1)
Changed lines of the file:
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@@
     (tracks 16)
     (zones 0)
-    (modules 8)
+    (modules 9)
     (nets 7)
   )
@@
     )
   )
+  (module OSHW_COPPER_10MM (layer F.Cu)
+    (at 30.48 19.05)
+    (fp_text reference OSHW_LOGO (at 0 6.35) (layer F.SilkS) hide
+      (effects (font (size 1.524 1.524) (thickness 0.3048)))
+    )
+    (fp_text value "" (at 2.54 8.89) (layer F.SilkS) hide
+      (effects (font (size 1.524 1.524) (thickness 0.3048)))
+    )
+    (pad "" smd trapezoid (at 0 -4.1656 180) (size 1.45796 1.4986) (rect_delta 0 -0.2794 )
+      (layers F.Cu F.Paste F.Mask)
+    )
+    (pad "" smd trapezoid (at 2.94386 -2.94386 135) (size 1.45796 1.4986) (rect_delta 0 -0.2794 )
+      (layers F.Cu F.Paste F.Mask)
+    )
+    (pad "" smd trapezoid (at 4.1656 0 90) (size 1.45796 1.4986) (rect_delta 0 -0.2794 )
+      (layers F.Cu F.Paste F.Mask)
+    )
+    (pad "" smd trapezoid (at 2.94386 2.94386 45) (size 1.45796 1.4986) (rect_delta 0 -0.2794 )
+      (layers F.Cu F.Paste F.Mask)
+    )
+    (pad "" smd trapezoid (at -2.94386 -2.94386 225) (size 1.45796 1.4986) (rect_delta 0 -0.2794 )
+      (layers F.Cu F.Paste F.Mask)
+    )
+    (pad "" smd trapezoid (at -4.1656 0 270) (size 1.45796 1.4986) (rect_delta 0 -0.2794 )
+      (layers F.Cu F.Paste F.Mask)
+    )
+    (pad "" smd trapezoid (at -2.94386 2.94386 315) (size 1.45796 1.4986) (rect_delta 0 -0.2794 )
+      (layers F.Cu F.Paste F.Mask)
+    )
+    (pad "" smd trapezoid (at 0 -2.39522 180) (size 1.08204 2.29108) (rect_delta 0 0.41402 )
+      (layers F.Cu F.Paste F.Mask)
+    )
+    (pad "" smd trapezoid (at -0.9144 -2.21234 202.5) (size 1.08204 2.29108) (rect_delta 0 0.41402 )
+      (layers F.Cu F.Paste F.Mask)
+    )
+    (pad "" smd trapezoid (at 0.9144 -2.21234 157.5) (size 1.08204 2.29108) (rect_delta 0 0.41402 )
+      (layers F.Cu F.Paste F.Mask)
+    )
+    (pad "" smd trapezoid (at 1.69164 -1.69164 135) (size 1.08204 2.29108) (rect_delta 0 0.41402 )
+      (layers F.Cu F.Paste F.Mask)
+    )
+    (pad "" smd trapezoid (at -1.69164 -1.69164 225) (size 1.08204 2.29108) (rect_delta 0 0.41402 )
+      (layers F.Cu F.Paste F.Mask)
+    )
+    (pad "" smd trapezoid (at 2.21234 -0.9144 112.5) (size 1.08204 2.29108) (rect_delta 0 0.41402 )
+      (layers F.Cu F.Paste F.Mask)
+    )
+    (pad "" smd trapezoid (at -2.21234 -0.9144 247.5) (size 1.08204 2.29108) (rect_delta 0 0.41402 )
+      (layers F.Cu F.Paste F.Mask)
+    )
+    (pad "" smd trapezoid (at 2.39522 0 90) (size 1.08204 2.29108) (rect_delta 0 0.41402 )
+      (layers F.Cu F.Paste F.Mask)
+    )
+    (pad "" smd trapezoid (at -2.39522 0 270) (size 1.08204 2.29108) (rect_delta 0 0.41402 )
+      (layers F.Cu F.Paste F.Mask)
+    )
+    (pad "" smd trapezoid (at -2.21234 0.9144 292.5) (size 1.08204 2.29108) (rect_delta 0 0.41402 )
+      (layers F.Cu F.Paste F.Mask)
+    )
+    (pad "" smd trapezoid (at 2.21234 0.9144 67.5) (size 1.08204 2.29108) (rect_delta 0 0.41402 )
+      (layers F.Cu F.Paste F.Mask)
+    )
+    (pad "" smd trapezoid (at 1.69164 1.69164 45) (size 1.08204 2.29108) (rect_delta 0 0.41402 )
+      (layers F.Cu F.Paste F.Mask)
+    )
+    (pad "" smd trapezoid (at -1.69164 1.69164 315) (size 1.08204 2.29108) (rect_delta 0 0.41402 )
+      (layers F.Cu F.Paste F.Mask)
+    )
+    (pad "" smd trapezoid (at -1.32842 1.99136 326.3) (size 0.54102 2.29108) (rect_delta 0 0.20828 )
+      (layers F.Cu F.Paste F.Mask)
+    )
+    (pad "" smd trapezoid (at 1.32842 1.99136 33.7) (size 0.54102 2.29108) (rect_delta 0 0.20828 )
+      (layers F.Cu F.Paste F.Mask)
+    )
+  )
